Commit message: feat: 接入头部控制与关节空间复位, 运动学切换为预编译 SO 交付
- bw_std_control: 新增 StandardHeadController 与 arm_power_on_sequence 分阶段上电, 命令安全补充头部边界与夹爪零位容差, 协议命名去除 V3 前缀.
- bw_kinematics: 新增 Algorithm Provider 支持预编译 SO 与源码两种交付, 公共接口收敛并隐藏 Pinocchio/CasADi 类型, 新增 standard_ik.urdf 资产与 Ruckig 在线平滑.
- bw_teleop: 复位改由 /kinematics/reset_arms 下发关节空间斜坡, 新增 /teleop/control_active 映射 safety/power, 头部增加零参考与恢复后 re-anchor, 支持单手操作.
- bw_std_description / bw_std_bringup: ros2_control 补齐 head command-only GPIO 与 17 关节契约, head_controller 接入启动与参数传递.
- scripts: 新增 tmux 托管的 start.sh, 支持 real/readonly/mock 三种放行模式, 启动前检查 session、遗留进程与串口占用.
- docs: 精简根与各包 README, 去除重复说明, 更新启动流程与 Mock/真机验证命令.
- 移除各包测试与本包源码级算法依赖.

File: src/bw_std_description/urdf/standard.ros2_control.xacro (robot description, xacro)
@@ -1,5 +1,5 @@
 <?xml version="1.0"?>
 <robot xmlns:xacro="http://www.ros.org/wiki/xacro">
-  <!-- 受控关节使用统一接口，真机和 mock 因此具有相同的控制器契约。 -->
+  <!-- 受控关节使用统一接口-->
   <xacro:macro name="standard_position_joint" params="joint_name lower upper initial_value:=0.0">
     <joint name="${joint_name}">
@@ -16,5 +16,5 @@
   </xacro:macro>
   <xacro:macro name="standard_ros2_control"
-               params="name use_mock_hardware serial_port baud_rate feedback_timeout_ms power_on_on_activate arm_mapping_calibrated left_arm_motor_indices right_arm_motor_indices left_arm_direction right_arm_direction left_arm_raw_zero_rad right_arm_raw_zero_rad arm_max_velocity_rad_s pelvis_max_velocity_mm_s gripper_max_velocity_normalized_s">
+               params="name use_mock_hardware serial_port baud_rate feedback_timeout_ms power_on_on_activate arm_mapping_calibrated left_arm_motor_indices right_arm_motor_indices left_arm_direction right_arm_direction left_arm_raw_zero_rad right_arm_raw_zero_rad arm_max_velocity_rad_s pelvis_max_velocity_mm_s gripper_max_velocity_normalized_s arm_startup_limit_tolerance_rad gripper_startup_limit_tolerance_m head_max_velocity_rad_s command_rate_hz">
     <ros2_control name="${name}" type="system">
       <hardware>
@@ -39,4 +39,8 @@
           <param name="pelvis_max_velocity_mm_s">${pelvis_max_velocity_mm_s}</param>
           <param name="gripper_max_velocity_normalized_s">${gripper_max_velocity_normalized_s}</param>
+          <param name="arm_startup_limit_tolerance_rad">${arm_startup_limit_tolerance_rad}</param>
+          <param name="gripper_startup_limit_tolerance_m">${gripper_startup_limit_tolerance_m}</param>
+          <param name="head_max_velocity_rad_s">${head_max_velocity_rad_s}</param>
+          <param name="command_rate_hz">${command_rate_hz}</param>
         </xacro:unless>
       </hardware>
@@ -61,8 +65,8 @@
       <xacro:standard_position_joint
         joint_name="C_joint"
-        lower="-0.231"
-        upper="0.231"
-        initial_value="0.0"/>
-      <!-- 真机与 mock 共用机体速度 GPIO，不导出虚构的轮关节反馈。 -->
+        lower="-0.5"
+        upper="0.0"
+        initial_value="-0.1"/>
+      <!-- 真机与 mock 共用机体速度 GPIO -->
       <gpio name="base">
         <command_interface name="vx"/>
@@ -70,4 +74,26 @@
         <command_interface name="wz"/>
       </gpio>
+      <!-- 头部导出 command-only GPIO -->
+      <gpio name="head">
+        <command_interface name="pitch">
+          <param name="min">-0.524</param>
+          <param name="max">0.785</param>
+        </command_interface>
+        <command_interface name="yaw">
+          <param name="min">-1.570</param>
+          <param name="max">1.570</param>
+        </command_interface>
+        <command_interface name="roll">
+          <param name="min">-0.349</param>
+          <param name="max">0.349</param>
+        </command_interface>
+      </gpio>
+      <!-- 安全 GPIO: 遥操作控制活跃请求 1; VR 断流后请求 0 触发软件掉电。 -->
+      <gpio name="safety">
+        <command_interface name="power">
+          <param name="min">0</param>
+          <param name="max">1</param>
+        </command_interface>
+      </gpio>
     </ros2_control>
   </xacro:macro>

File: src/bw_std_description/urdf/standard.urdf (robot description, URDF)
Before this commit: robot standard, 27 links, 26 joints
Joints:
- joint C_joint: limit lower=-0.231 upper=0.231 effort=100 velocity=0.02 -> lower=-0.5 upper=0.0 effort=100 velocity=0.02

File: src/bw_std_description/urdf/standard.xacro (robot description, xacro)
@@ -16,4 +16,8 @@
   <xacro:arg name="pelvis_max_velocity_mm_s" default="20.0"/>
   <xacro:arg name="gripper_max_velocity_normalized_s" default="0.2"/>
+  <xacro:arg name="arm_startup_limit_tolerance_rad" default="0"/>
+  <xacro:arg name="gripper_startup_limit_tolerance_m" default="0"/>
+  <xacro:arg name="head_max_velocity_rad_s" default="1.0"/>
+  <xacro:arg name="command_rate_hz" default="200.0"/>
   <xacro:include filename="standard.urdf"/>
   <xacro:include filename="standard.ros2_control.xacro"/>
@@ -34,4 +38,8 @@
     arm_max_velocity_rad_s="$(arg arm_max_velocity_rad_s)"
     pelvis_max_velocity_mm_s="$(arg pelvis_max_velocity_mm_s)"
-    gripper_max_velocity_normalized_s="$(arg gripper_max_velocity_normalized_s)"/>
+    gripper_max_velocity_normalized_s="$(arg gripper_max_velocity_normalized_s)"
+    arm_startup_limit_tolerance_rad="$(arg arm_startup_limit_tolerance_rad)"
+    gripper_startup_limit_tolerance_m="$(arg gripper_startup_limit_tolerance_m)"
+    head_max_velocity_rad_s="$(arg head_max_velocity_rad_s)"
+    command_rate_hz="$(arg command_rate_hz)"/>
 </robot>
