Commit message: chore(bw_std_bringup): 同步双臂第4关节上限
- 将左右臂第4关节上限从 1.355 rad 调整为 1.45 rad.
- 同步 URDF 模型与 ros2_control 限位定义.
- 保持关节下限及其他参数不变.

File: src/bw_std_bringup/urdf/standard.ros2_control.xacro (robot description, xacro)
@@ -49,5 +49,5 @@
       <xacro:standard_position_joint joint_name="A_left_Degree2_joint" lower="-0.142" upper="2.077"/>
       <xacro:standard_position_joint joint_name="A_left_Degree3_joint" lower="-1.541" upper="1.541"/>
-      <xacro:standard_position_joint joint_name="A_left_Degree4_joint" lower="-0.529" upper="1.355"/>
+      <xacro:standard_position_joint joint_name="A_left_Degree4_joint" lower="-0.529" upper="1.45"/>
       <xacro:standard_position_joint joint_name="A_left_Degree5_joint" lower="-1.540" upper="1.540"/>
       <xacro:standard_position_joint joint_name="A_left_Degree6_joint" lower="-0.756" upper="0.756"/>
@@ -56,5 +56,5 @@
       <xacro:standard_position_joint joint_name="A_right_Degree2_joint" lower="-2.077" upper="0.142"/>
       <xacro:standard_position_joint joint_name="A_right_Degree3_joint" lower="-1.541" upper="1.541"/>
-      <xacro:standard_position_joint joint_name="A_right_Degree4_joint" lower="-0.529" upper="1.355"/>
+      <xacro:standard_position_joint joint_name="A_right_Degree4_joint" lower="-0.529" upper="1.45"/>
       <xacro:standard_position_joint joint_name="A_right_Degree5_joint" lower="-1.540" upper="1.540"/>
       <xacro:standard_position_joint joint_name="A_right_Degree6_joint" lower="-0.756" upper="0.756"/>

File: src/bw_std_bringup/urdf/standard.urdf (robot description, URDF)
Before this commit: robot standard, 27 links, 26 joints
Joints:
- joint A_left_Degree4_joint: limit lower=-0.529 upper=1.355 effort=10 velocity=0.1 -> lower=-0.529 upper=1.45 effort=10 velocity=0.1
- joint A_right_Degree4_joint: limit lower=-0.529 upper=1.355 effort=10 velocity=0.1 -> lower=-0.529 upper=1.45 effort=10 velocity=0.1
